File: Schema_carte/ESP_CAM_VVN.sch (EAGLE design)
At the start: 50 parts, among them Q1 SI2305CDS, Q2 BSS131, Q4 BSS138, Q5 BSS138, Q6 SI2305CDS, Q7 BSS131, U1 MCP3428-E/SL, U2 ESP32-WROVER-E, U3 PCA9685PW, U5 MIC5239S, X1 B2B-PH-K-S, X2 FH12-24S-0.5SH

Commit message: romain maj
Parts:
- added R11: 10k, eagle-ltspice:RR1206
Connections:
- net N$9 renamed V2_1.8V
- removed net CA_RST: X2-6.1
- removed net SD_CMD: SD1.CMD
- net CA_PWDN: now also R11.2
- net CA_RST_SD_CMD: now also SD1.CMD, X2-6.1
- net GND: now also R11.1
Changed lines of the file:
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@@
 <part name="R9" library="eagle-ltspice" library_urn="urn:adsk.eagle:library:217" deviceset="R" device="R1206" package3d_urn="urn:adsk.eagle:package:13301/1" value="4.7K"/>
 <part name="R10" library="eagle-ltspice" library_urn="urn:adsk.eagle:library:217" deviceset="R" device="R1206" package3d_urn="urn:adsk.eagle:package:13301/1" value="4.7K"/>
+<part name="R11" library="eagle-ltspice" library_urn="urn:adsk.eagle:library:217" deviceset="R" device="R1206" package3d_urn="urn:adsk.eagle:package:13301/1" value="10k"/>
+<part name="SUPPLY24" library="supply2" library_urn="urn:adsk.eagle:library:372" deviceset="GND" device=""/>
 </parts>
 <sheets>
@@
 <attribute name="VALUE" x="210.82" y="72.898" size="1.778" layer="96"/>
 </instance>
+<instance part="R11" gate="G$1" x="212.09" y="68.58" smashed="yes">
+<attribute name="NAME" x="210.82" y="70.0786" size="1.778" layer="95"/>
+<attribute name="VALUE" x="210.82" y="65.278" size="1.778" layer="96"/>
+</instance>
+<instance part="SUPPLY24" gate="GND" x="204.47" y="68.58" smashed="yes" rot="R270"/>
 </instances>
 <busses>
@@
 <wire x1="195.58" y1="45.72" x2="193.04" y2="45.72" width="0.1524" layer="91"/>
 <pinref part="SUPPLY23" gate="GND" pin="GND"/>
+</segment>
+<segment>
+<pinref part="R11" gate="G$1" pin="1"/>
+<pinref part="SUPPLY24" gate="GND" pin="GND"/>
 </segment>
 </net>
@@
 </segment>
 </net>
-<net name="SD_CMD" class="0">
-<segment>
-<pinref part="SD1" gate="G$1" pin="CMD"/>
-<wire x1="146.05" y1="57.15" x2="140.97" y2="57.15" width="0.1524" layer="91"/>
-<label x="132.08" y="57.15" size="1.778" layer="95"/>
-</segment>
-</net>
 <net name="SD_CLK" class="0">
 <segment>
@@
 <label x="240.03" y="121.92" size="1.778" layer="95"/>
 </segment>
-</net>
-<net name="CA_RST" class="0">
 <segment>
 <pinref part="X2" gate="-6" pin="1"/>
 <wire x1="238.76" y1="73.66" x2="233.68" y2="73.66" width="0.1524" layer="91"/>
-<label x="228.6" y="73.66" size="1.778" layer="95"/>
+<label x="219.71" y="73.66" size="1.778" layer="95"/>
+</segment>
+<segment>
+<pinref part="SD1" gate="G$1" pin="CMD"/>
+<wire x1="146.05" y1="57.15" x2="140.97" y2="57.15" width="0.1524" layer="91"/>
+<label x="123.19" y="57.15" size="1.778" layer="95"/>
 </segment>
 </net>
@@
 <segment>
 <pinref part="X2" gate="-8" pin="1"/>
-<wire x1="238.76" y1="68.58" x2="233.68" y2="68.58" width="0.1524" layer="91"/>
+<wire x1="238.76" y1="68.58" x2="217.17" y2="68.58" width="0.1524" layer="91"/>
 <label x="228.6" y="68.58" size="1.778" layer="95"/>
-</segment>
-</net>
-<net name="N$9" class="0">
+<pinref part="R11" gate="G$1" pin="2"/>
+</segment>
+</net>
+<net name="V2_1.8V" class="0">
 <segment>
 <pinref part="X2" gate="-10" pin="1"/>
-<wire x1="238.76" y1="63.5" x2="203.2" y2="63.5" width="0.1524" layer="91"/>
+<wire x1="238.76" y1="63.5" x2="212.09" y2="63.5" width="0.1524" layer="91"/>
 <pinref part="C22" gate="G$1" pin="1"/>
-</segment>
-</net>
+<junction x="212.09" y="63.5"/>
+<wire x1="212.09" y1="63.5" x2="203.2" y2="63.5" width="0.1524" layer="91"/>
+<wire x1="212.09" y1="63.5" x2="212.09" y2="66.04" width="0.1524" layer="91"/>
+<wire x1="212.09" y1="66.04" x2="190.5" y2="66.04" width="0.1524" layer="91"/>
+<label x="186.69" y="67.31" size="1.778" layer="95"/>
+</segment>
+</net>

Commit message: romain
Parts:
- removed C21: 100n, eagle-ltspice:CC1206
- removed D1: DISPLAY-OLED-128X64-I2C1.3_BIS, diy-modules1.8-perso:DISPLAY-OLED-128X64-I2C1.3_BIS
- removed Q5: BSS138, detect:BSS138
- removed R28: 10k, eagle-ltspice:RR1206
- added C5, C6: 1u, rcl:C-EUC1210K
- added JP2, MOT: (no value), pinhead:PINHD-1X2
- added M1: ELECTRET_MICROPHON-WM-62PC/62PK, microphon:ELECTRET_MICROPHON-WM-62PC/62PK
- added Q3: SI2305CDS, transistor-small-signal-perso:SI2305CDS
- added Q8: BSS131, transistor-small-signal-perso:BSS131
- added R13: 100k, rcl:R-EU_R1206
- added R14: 220k, rcl:R-EU_R1206
- added R15: 12k, rcl:R-EU_R1206
- added R16: 10k, rcl:R-EU_R1206
- added R17, R18: 33k, eagle-ltspice:RR1206
- added R21: 10k, eagle-ltspice:RR1206
- added SJ1: (no value), jumper:SJ2W
- added U4, U6: MIC5239-ADJMM, micrel:MIC5239-ADJMM
- R20: value 27k -> 33k
- R4: value 0 -> 33k
Connections:
- removed net +12V: C12.1, C13.1, R19.1, U5.IN, X1.2
- removed net VBAT: R4.1
- new net +5V: C12.1, C13.1, Q3.S, R17.2, R19.1, U5.IN, X1.2
- new net +5V/1: Q3.D, R4.1, SJ1.1
- new net 5V_MES: R20.1, R4.2, U1.CH3+
- new net N$11: M1.2, R21.1, U1.CH1+
- new net N$12: JP2.1, U1.CH4-
- new net N$13: MOT.1, U3.LED0
- new net N$14: MOT.2, U3.LED1
- new net N$9: Q3.G, Q8.D, R17.1
- new net N$91: R13.1, R14.2, U6.ADJ
- new net N$92: R15.1, R16.2, U4.ADJ
- new net V1_2.7V: C5.1, R15.2, U4.OUT
- net GND: now also C5.2, C6.2, M1.1, Q8.S, R14.1, R16.1, R18.2, R20.2, U1.CH1-, U1.CH2-, U1.CH3-, U4.GND, U6.GND; no longer C21.2, D1.GND, R28.2
- net LDR: now also U1.CH2+
- net LED_G: now also U3.LED15
- net LED_R: now also U3.LED14
- net N$4: now also SJ1.2, U3.VDD; no longer C21.1, Q5.S, R28.1, R4.2
- net N$5: now also JP2.2, U1.CH4+; no longer Q5.D, R20.1
- net POWER: now also Q8.G, R18.1, U3.LED2; no longer Q5.G
- net POWER_SD: now also U3.LED3
- net SCL: no longer D1.SCL
- net SDA: no longer D1.SDA
- net V+: now also R21.2, SJ1.3, U4.EN, U4.IN, U6.EN, U6.IN; no longer D1.VCC, U3.VDD
- net V2_1.8V: now also C6.1, R13.2, U6.OUT
- net VCC: no longer R20.2
Other:
- note removed: "OLED display"
- moved on the sheet: C22, C4, Q6, Q7, R10, R11, R20, R4, R6, R7, R8, R9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
