File: Schema_carte/Final/ESP_CAM_VVN_v4.sch (EAGLE design)
At the start: 64 parts, among them M1 ELECTRET_MICROPHON-WM-62PC/62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, Q1 SI2305CDS, Q2 BSS131, Q3 SI2305CDS, Q4 BSS138, Q6 SI2305CDS, Q7 BSS131, Q8 BSS131, U1 MCP3428-E/SL, U2 ESP32-WROVER-E, U3 PCA9685PW, U4 MIC5239-ADJMM, U5 MIC5239S, U6 MIC5239-ADJMM, X1 B2B-PH-K-S, X2 FH12-24S-0.5SH

Commit message: romain maj
Parts:
- removed JP1: (no value), pinhead:PINHD-1X4
- removed JP2: (no value), pinhead:PINHD-1X2
- removed OPH1: VT93N2, photo-elements:VT93N2
- removed Q4: BSS138, detect:BSS138
- removed R18, R20, R4: 33k, eagle-ltspice:RR1206
- removed SJ1: (no value), jumper:SJ2W
- added /OE, OUTPUTS: (no value), jumper:SJ2W
- added C7, C8: 100n, eagle-ltspice:CC1206
- added CAN, WAKEUP: (no value), pinhead:PINHD-1X2
- added I2C: (no value), pinhead:PINHD-1X4
- added LDR: VT93N2, photo-elements:VT93N2
- added R26: 100k, eagle-ltspice:RR1206
- added S: (no value), pinhead:PINHD-1X6
- C12, C14, C2: device eagle-ltspice:CC1210 -> eagle-ltspice:CC1206
- C5, C6: device rcl:C-EUC1210K -> rcl:C-EUC1206
- JP6: device pinhead:PINHD-1X6 -> pinhead:PINHD-1X6/90
- MOT: device pinhead:PINHD-1X2 -> pinhead:PINHD-1X4
Connections:
- net N$13 renamed M1
- removed net N$14: MOT.2, U3.LED1
- removed net N$2: Q4.D, R19.2
- removed net V1_2.5V: X2-4.1
- removed net VALIM: R3.1
- new net M2: MOT.3, U3.LED1
- new net N$15: S.1, U3.LED8
- new net N$16: S.2, U3.LED9
- new net N$17: S.3, U3.LED10
- new net N$18: S.4, U3.LED11
- new net N$19: S.5, U3.LED12
- new net N$20: S.6, U3.LED13
- new net OE: /OE.2, U3./OE
- net +5V: no longer R19.1
- net +5V/1: now also OUTPUTS.1, R19.1; no longer R4.1, SJ1.1
- net 5V_MES: now also R3.1; no longer R20.1, R4.2
- net GND: now also /OE.1, C7.2, C8.2, I2C.4, LDR.1, MOT.2, MOT.4, U1.ADR0, U1.ADR1, U1.VSS, U3.A0, U3.A1, U3.A2, U3.A3, U3.A4, U3.A5, U3.EXTCLK, WAKEUP.1; no longer JP1.4, LED_G.C, LED_R.C, OPH1.1, R18.2, R20.2
- net LDR: now also LDR.2; no longer OPH1.2
- net N$12: now also CAN.1; no longer JP2.1
- net N$3: now also R19.2; no longer Q4.S
- net N$4: now also /OE.3, C8.1, LED_G.A, LED_R.A, OUTPUTS.2; no longer SJ1.2
- net N$5: now also CAN.2; no longer JP2.2
- net N$7: now also LED_R.C; no longer LED_R.A
- net N$8: now also LED_G.C; no longer LED_G.A
- net POWER: no longer Q4.G, R18.1
- net SCL: now also I2C.2; no longer JP1.2
- net SDA: now also I2C.3; no longer JP1.3
- net SD_D3: now also R26.2, WAKEUP.2
- net V+: now also C7.1, I2C.1, OUTPUTS.3; no longer JP1.1, SJ1.3
- net V1_2.7V: now also X2-4.1
- net VCC: now also R26.1
Other:
- note added: "V 4.0"
- note removed: "V ?????"
- moved on the sheet: C5, C6, LED_G, LED_R, Q1, Q3, R13, R14, R15, R16, R17, R22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
