File: Schema_carte/Final/ESP_CAM_VVN_v5.sch (EAGLE design)
At the start: 66 parts, among them M1 ELECTRET_MICROPHON-WM-62PC/62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, Q1 SI2305CDS, Q2 BSS131, Q3 SI2305CDS, Q6 SI2305CDS, Q7 BSS131, Q8 BSS131, U1 MCP3428-E/SL, U2 ESP32-WROVER-E, U3 PCA9685PW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

Commit message: romain maj
Parts:
- removed M1: ELECTRET_MICROPHON-WM-62PC/62PK, microphon:ELECTRET_MICROPHON-WM-62PC/62PK
- added AR, GAIN: (no value), jumper:SJ2W
- added MAX9814: (no value), pinhead:PINHD-1X5
- added R18, R20, R27, R4: 47k, rcl:R-EU_R0805
- added SD_SPI: (no value), pinhead:PINHD-1X6
- R21: value 10k -> 47k; device eagle-ltspice:RR1206 -> rcl:R-EU_R0805
Connections:
- removed net N$11: M1.2, R21.1, U1.CH1+
- removed net SD_CLK: SD1.VDD
- new net AR: AR.2, MAX9814.1
- new net GAIN: GAIN.2, MAX9814.3
- new net N$2: MAX9814.2, U1.CH1+
- net +5V: now also OUTPUTS.1
- net +5V/1: no longer OUTPUTS.1
- net CA_D0_SD_D1: now also R20.2
- net CA_PWDN_SD_CLK: now also SD1.VDD, SD_SPI.4
- net CA_RST_SD_CMD: now also R27.2
- net GND: now also AR.3, GAIN.1, MAX9814.5, SD_SPI.6; no longer M1.1
- net IO0: now also U2.IO0
- net RX: now also U2.RXD0; no longer U2.TXD0
- net SD_D0: now also R21.2, SD_SPI.2
- net SD_D2: now also R18.2, SD_SPI.3
- net SD_D3: now also R4.2, SD_SPI.5
- net TX: now also U2.TXD0; no longer U2.RXD0
- net V+: now also AR.1, GAIN.3, MAX9814.4; no longer OUTPUTS.3, R21.2
- net V+_SD: now also R18.1, R20.1, R21.1, R27.1, R4.1, SD_SPI.1
- net VCC: now also OUTPUTS.3
Other:
- note added: "V 5.1"
- note removed: "V 4.0"
- moved on the sheet: I2C, R21
